File: kicad/_saved_z80.sch (KiCad schematic (older format))
At the start: 23 parts, among them SW1 SW_PUSH, U1 Z80CPU, U2 z80pcb, U3 74HC14

Commit message: fixed connections
Parts:
- U4: renamed from U?; footprint (none) -> Housings_DIP:DIP-16_W7.62mm
Changed lines of the file:
@@
 LIBS:valves
 LIBS:Zilog
+LIBS:Oscillators
+LIBS:cmos_ieee
 LIBS:z80-cache
 EELAYER 25 0
@@
 	10050 4700 10700 4700
 Wire Wire Line
-	7850 4400 9100 4400
+	7850 4400 8700 4400
 Wire Wire Line
 	8550 4400 8550 5050
@@
 	9400 4800 9400 5600
 Wire Wire Line
-	5400 5600 11100 5600
+	5400 5600 10700 5600
 Wire Wire Line
 	7550 3400 7450 3400
 Connection ~ 7450 3400
 Wire Wire Line
-	7850 3400 9100 3400
-Wire Wire Line
-	7850 2800 9100 2800
-Wire Wire Line
-	7850 2700 9100 2700
+	7850 2800 8700 2800
 Wire Wire Line
 	7850 2700 7850 2650
@@
 Connection ~ 5400 3200
 $Comp
-L 74LS163 U?
+L 74LS163 U4
 U 1 1 5728B2B4
 P 2450 5000
-F 0 "U?" H 2500 5100 50  0000 C CNN
+F 0 "U4" H 2500 5100 50  0000 C CNN
 F 1 "74LS163" H 2550 4800 50  0000 C CNN
-F 2 "" H 2450 5000 50  0000 C CNN
+F 2 "Housings_DIP:DIP-16_W7.62mm" H 2450 5000 50  0000 C CNN
 F 3 "" H 2450 5000 50  0000 C CNN
 	1    2450 5000
@@
 $EndComp
 $Comp
-L +5V #PWR?
+L +5V #PWR03
 U 1 1 5728BB0F
 P 1400 4350
-F 0 "#PWR?" H 1400 4200 50  0001 C CNN
+F 0 "#PWR03" H 1400 4200 50  0001 C CNN
 F 1 "+5V" H 1400 4490 50  0000 C CNN
 F 2 "" H 1400 4350 50  0000 C CNN
@@
 	1750 5000 1400 5000
 Connection ~ 1400 5000
+Wire Wire Line
+	7850 3400 8700 3400
+Wire Wire Line
+	7850 2700 8700 2700
 $EndSCHEMATC
