File: kicad/z80.kicad_pcb (KiCad board)
At the start: 2 copper layers, 17 parts, among them U1 Z80CPU, U2 z80pcb

Commit message: add reset circuit
Parts:
- added C2: 47μF, Capacitors_ThroughHole:C_Radial_D7.5_L11.2_P2.5, F.Cu at (202.6, 103.5)
- added D6: 1N4148, Diodes_ThroughHole:Diode_DO-35_SOD27_Horizontal_RM10, F.Cu at (186.7, 103.5)
- added R10: 10k, Resistors_ThroughHole:Resistor_Horizontal_RM10mm, F.Cu at (186.7, 107.3)
- added SW1: SW_PUSH, kicad:vintage_reset, F.Cu at (191.8, 117.5)
- added U3: 74HC14, Housings_DIP:DIP-14_W7.62mm, F.Cu at (174.0, 107.3)
Connections:
- net Net-(C1-Pad1) renamed VCC
- C1 pad 2: Net-(C1-Pad2) -> GND
- D1 pad 1: Net-(C1-Pad2) -> GND
- D2 pad 1: Net-(C1-Pad2) -> GND
- D3 pad 1: Net-(C1-Pad2) -> GND
- D4 pad 1: Net-(C1-Pad2) -> GND
- D5 pad 1: Net-(C1-Pad2) -> GND
- U1 pad 16: Net-(R4-Pad2) -> Net-(U1-Pad16)
- U1 pad 17: Net-(R3-Pad2) -> Net-(U1-Pad17)
- U1 pad 18: Net-(R2-Pad2) -> Net-(U1-Pad18)
- U1 pad 25: Net-(R1-Pad2) -> Net-(U1-Pad25)
- U1 pad 29: Net-(C1-Pad2) -> GND
- U2 pad 29: Net-(C1-Pad2) -> Net-(U2-Pad29)
Routing:
- net GND: track 0.00 -> 202.6 mm
- net Net-(C1-Pad2): track 122.0 -> 0.00 mm
- net VCC: track 102.4 -> 162.3 mm
- net Net-(C2-Pad1): track 0.00 -> 56.3 mm, vias 0 -> 2
- net Net-(U1-Pad26): track 26.3 -> 74.7 mm, vias 0 -> 2
- net Net-(U2-Pad29): track 0.00 -> 23.0 mm
- net Net-(R4-Pad2): track 35.3 -> 20.1 mm
- net Net-(U1-Pad16): track 0.00 -> 15.2 mm
- net Net-(R3-Pad2): track 35.4 -> 22.7 mm
- net Net-(U1-Pad17): track 0.00 -> 12.7 mm
- net Net-(U3-Pad2): track 0.00 -> 2.54 mm
- net Net-(U1-Pad25): track 0.00 -> 1.71 mm
- net Net-(R1-Pad2): track 33.4 -> 31.7 mm

Commit message: fixed connections
Parts:
- added U4: 74LS163, Housings_DIP:DIP-16_W7.62mm, F.Cu at (172.7, 62.9)
- moved U3 3.81 mm to (174.0, 111.1)
- moved D5 3.17 mm to (104.1, 67.3)
- moved U2 3.17 mm to (141.0, 93.3)
- moved C1 2.01 mm to (109.9, 85.7), turned to 270 degrees
- moved R9 1.27 mm to (106.7, 82.5)
Connections:
- U1 pad 16: Net-(U1-Pad16) -> Net-(R4-Pad2)
- U1 pad 17: Net-(U1-Pad17) -> Net-(R3-Pad2)
- U1 pad 18: Net-(U1-Pad18) -> Net-(R2-Pad2)
- U1 pad 25: Net-(U1-Pad25) -> Net-(R1-Pad2)
- U2 pad 29: Net-(U2-Pad29) -> GND
Routing:
- net GND: track 202.6 -> 264.3 mm, vias 0 -> 2
- net VCC: track 162.3 -> 214.8 mm
- net Net-(U2-Pad29): track 23.0 -> 0.00 mm
- net Net-(U1-Pad16): track 15.2 -> 0.00 mm
- net Net-(R4-Pad2): track 20.1 -> 34.7 mm
- net Net-(U1-Pad17): track 12.7 -> 0.00 mm
- net Net-(R3-Pad2): track 22.7 -> 34.8 mm
- net Net-(U1-Pad26): track 74.7 -> 80.6 mm
- net Net-(R1-Pad2): track 31.7 -> 36.4 mm
- net Net-(R7-Pad1): track 46.9 -> 50.5 mm
- net Net-(U1-Pad40): track 26.7 -> 29.9 mm
- net Net-(U1-Pad39): track 26.7 -> 29.9 mm
- net Net-(U1-Pad38): track 26.7 -> 29.9 mm
- net Net-(U1-Pad37): track 26.7 -> 29.9 mm
- net Net-(U1-Pad36): track 26.7 -> 29.9 mm
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Other:
- net class Default: clearance 0.2 -> 0.1
- net class GND added: clearance 0.1, trace_width 0.6, via_dia 1.52, via_drill 0.76
- rule trace_clearance: 0.2 -> 0.1

Commit message: finish cpu board draft
Parts:
- added C3: 10μF, Capacitors_ThroughHole:C_Radial_D7.5_L11.2_P2.5, F.Cu at (204.5, 75.6)
- added D7: 1N4148, Diodes_ThroughHole:Diode_DO-35_SOD27_Horizontal_RM10, F.Cu at (181.6, 95.9)
- added P1: USB_B, Connect:USB_B, F.Cu at (199.4, 62.9)
- added R11: 10k, Resistors_ThroughHole:Resistor_Horizontal_RM10mm, F.Cu at (184.2, 95.9)
- added SW2: SW_PUSH, kicad:vintage_reset, F.Cu at (191.8, 90.8)
- added X1: 16.000Mhz, Oscillators:KXO-200_LargePads, F.Cu at (186.7, 70.5)
- U3: value 74HC14 -> 74LS132
- moved U4 25.7 mm to (176.5, 88.3), turned to 180 degrees
- moved U3 2.54 mm to (174.0, 108.6)
- moved D4 2.29 mm to (102.9, 98.4)
- moved C2 1.91 mm to (204.5, 103.5)
- moved R9 1.42 mm to (105.4, 83.2)
- moved D1 1.42 mm to (102.9, 121.3)
- moved D3 1.42 mm to (102.9, 106.0)
- moved D2 1.42 mm to (102.9, 113.7)
- moved D5 1.42 mm to (102.9, 67.9)
- moved SW1 1.27 mm to (191.8, 118.7)
- moved R1 1.27 mm to (135.9, 98.4)
- moved R10 1.27 mm to (186.7, 106.0)
- moved C1 0.63 mm to (110.5, 85.7)
Connections:
- U1 pad 6: Net-(U1-Pad6) -> CLOCK
- U2 pad 46: (no net) -> Net-(U2-Pad46)
- U2 pad 47: (no net) -> Net-(U2-Pad47)
- U2 pad 6: Net-(U1-Pad6) -> CLOCK
- U3 pad 10: (no net) -> Net-(U2-Pad47)
- U3 pad 11: (no net) -> Net-(U2-Pad47)
- U3 pad 12: (no net) -> Net-(C3-Pad1)
- U3 pad 13: (no net) -> Net-(C3-Pad1)
- U3 pad 2: Net-(U3-Pad2) -> Net-(C3-Pad1)
- U3 pad 3: Net-(U3-Pad2) -> Net-(U3-Pad3)
- U3 pad 4: Net-(U1-Pad26) -> Net-(U3-Pad3)
- U3 pad 5: (no net) -> Net-(U3-Pad3)
- U3 pad 6: (no net) -> Net-(U1-Pad26)
- U3 pad 8: (no net) -> Net-(U2-Pad46)
- U3 pad 9: (no net) -> Net-(U2-Pad47)
- U4 pad 10: Net-(U4-Pad10) -> VCC
- U4 pad 13: Net-(U4-Pad13) -> CLOCK
- U4 pad 3: Net-(U4-Pad3) -> GND
- U4 pad 4: Net-(U4-Pad4) -> GND
- U4 pad 5: Net-(U4-Pad5) -> GND
- U4 pad 6: Net-(U4-Pad6) -> GND
- U4 pad 7: Net-(U4-Pad7) -> VCC
Routing:
- net GND: track 264.3 -> 428.3 mm
- net VCC: track 214.8 -> 312.7 mm, vias 2 -> 4
- net Net-(C3-Pad1): track 0.00 -> 63.7 mm, vias 0 -> 2
- net CLOCK: track 0.00 -> 53.2 mm, vias 0 -> 6
- net Net-(U1-Pad6): track 32.8 -> 0.00 mm
- net Net-(U4-Pad2): track 0.00 -> 31.8 mm, vias 0 -> 1
- net Net-(U2-Pad47): track 0.00 -> 18.8 mm
- net Net-(C2-Pad1): track 54.2 -> 66.5 mm
- net Net-(U2-Pad46): track 0.00 -> 8.67 mm
- net Net-(U1-Pad26): track 80.6 -> 87.4 mm
- net Net-(U3-Pad3): track 0.00 -> 5.08 mm
- net Net-(U4-Pad14): track 0.00 -> 2.54 mm, vias 0 -> 1
- net Net-(U4-Pad12): track 0.00 -> 2.54 mm, vias 0 -> 1
- net Net-(U4-Pad11): track 0.00 -> 2.54 mm, vias 0 -> 1
- net Net-(U3-Pad2): track 2.54 -> 0.00 mm
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