File: kicad/z80uart/z80uart.sch (KiCad schematic (older format))
At the start: 4 parts

Commit message: add uart
Parts:
- added C1, C2: 100nF, Capacitors_ThroughHole:C_Disc_D3_P2.5, symbol C
- added U100: serial_port_interface, kicad:serial_to_usb_large, symbol serial_bort_interface
- U1: renamed from U?; footprint DIP-40 -> Housings_DIP:DIP-40_W15.24mm
- U101: renamed from U?; footprint (none) -> kicad:z80systemboard
- U2: renamed from U?; value 74LS138 -> 74LS238; footprint (none) -> Housings_DIP:DIP-16_W7.62mm
- X1: renamed from X?; footprint (none) -> Oscillators:KXO-200
Connections:
- net GND: now also U1.20 (GND), U101.29 (GND), C1.2, C2.2, U100.1 (GND)
- net VCC: now also U1.25 (~ADS~), U1.40 (VCC), C1.1, C2.1; no longer U2.6 (E3)
- net a7: now also U2.6 (E3); no longer U2.4 (E1)
- net uart_cs: now also U2.15 (O0); no longer U2.14 (O1)
- net iorq: now reaches U101.20 (IORQ)
- net iorq: now also U2.4 (E1)
- net rx: now reaches U1.10 (SIN)
- net rx: now also U100.4 (Rx)
- net tx: now reaches U1.11 (SOUT)
- net tx: now also U100.5 (Tx)
- net dtr: now reaches U1.33 (~DTR~)
- net dtr: now also U100.6 (DTR_Reset)
- net cts: now reaches U1.36 (~CTS~)
- net cts: now also U100.2 (CTS)
Changed lines of the file:
@@
 $EndDescr
 $Comp
-L z80pcb U?
+L z80pcb U101
 U 1 1 576A08A0
 P 10850 3440
-F 0 "U?" H 10850 3440 60  0000 C CNN
+F 0 "U101" H 10850 3440 60  0000 C CNN
 F 1 "z80pcb" H 10850 3440 60  0000 C CNN
-F 2 "" H 10850 3440 60  0000 C CNN
+F 2 "kicad:z80systemboard" H 10850 3440 60  0000 C CNN
 F 3 "" H 10850 3440 60  0000 C CNN
 	1    10850 3440
@@
 $EndComp
 $Comp
-L 16550 U?
+L 16550 U1
 U 1 1 576A0977
 P 6000 3760
-F 0 "U?" H 5150 5360 50  0000 L CNN
+F 0 "U1" H 5150 5360 50  0000 L CNN
 F 1 "16550" H 6600 5360 50  0000 L CNN
-F 2 "DIP-40" H 6000 3760 50  0000 C CIN
+F 2 "Housings_DIP:DIP-40_W15.24mm" H 6000 3760 50  0000 C CIN
 F 3 "" H 6000 3760 50  0000 C CNN
 	1    6000 3760
@@
 a2
 $Comp
-L 74LS138 U?
+L 74LS138 U2
 U 1 1 576A0D11
 P 8580 2630
-F 0 "U?" H 8680 3130 50  0000 C CNN
-F 1 "74LS138" H 8730 2081 50  0000 C CNN
-F 2 "" H 8580 2630 50  0000 C CNN
+F 0 "U2" H 8680 3130 50  0000 C CNN
+F 1 "74LS238" H 8730 2081 50  0000 C CNN
+F 2 "Housings_DIP:DIP-16_W7.62mm" H 8580 2630 50  0000 C CNN
 F 3 "" H 8580 2630 50  0000 C CNN
 	1    8580 2630
 	1    0    0    -1
 $EndComp
-Text GLabel 7980 2980 0    60   Input ~ 0
+Text GLabel 7980 2780 0    60   Input ~ 0
 a7
 Text GLabel 7980 2880 0    60   Input ~ 0
@@
 a7
 $Comp
-L VCC #PWR?
-U 1 1 576A1041
-P 7980 2780
-F 0 "#PWR?" H 7980 2630 50  0001 C CNN
-F 1 "VCC" H 7980 2930 50  0000 C CNN
-F 2 "" H 7980 2780 50  0000 C CNN
-F 3 "" H 7980 2780 50  0000 C CNN
-	1    7980 2780
-	1    0    0    -1
-$EndComp
-$Comp
-L VCC #PWR?
+L VCC #PWR01
 U 1 1 576A10B7
 P 10150 1040
-F 0 "#PWR?" H 10150 890 50  0001 C CNN
+F 0 "#PWR01" H 10150 890 50  0001 C CNN
 F 1 "VCC" H 10150 1190 50  0000 C CNN
 F 2 "" H 10150 1040 50  0000 C CNN
@@
 $EndComp
 $Comp
-L GND #PWR?
+L GND #PWR02
 U 1 1 576A1322
-P 10160 5840
-F 0 "#PWR?" H 10160 5590 50  0001 C CNN
-F 1 "GND" H 10160 5690 50  0000 C CNN
-F 2 "" H 10160 5840 50  0000 C CNN
-F 3 "" H 10160 5840 50  0000 C CNN
-	1    10160 5840
-	1    0    0    -1
-$EndComp
-Text GLabel 9180 2380 2    60   Input ~ 0
+P 10150 5840
+F 0 "#PWR02" H 10150 5590 50  0001 C CNN
+F 1 "GND" H 10150 5690 50  0000 C CNN
+F 2 "" H 10150 5840 50  0000 C CNN
+F 3 "" H 10150 5840 50  0000 C CNN
+	1    10150 5840
+	1    0    0    -1
+$EndComp
+Text GLabel 9180 2280 2    60   Input ~ 0
 uart_cs
 Text GLabel 5000 3760 0    60   Input ~ 0
 uart_cs
 $Comp
-L VCC #PWR?
-U 1 1 576A1B73
-P 4790 3560
-F 0 "#PWR?" H 4790 3410 50  0001 C CNN
-F 1 "VCC" H 4790 3710 50  0000 C CNN
-F 2 "" H 4790 3560 50  0000 C CNN
-F 3 "" H 4790 3560 50  0000 C CNN
-	1    4790 3560
-	1    0    0    -1
-$EndComp
-$Comp
-L VCC #PWR?
-U 1 1 576A1DB5
-P 4730 3660
-F 0 "#PWR?" H 4730 3510 50  0001 C CNN
-F 1 "VCC" H 4730 3810 50  0000 C CNN
-F 2 "" H 4730 3660 50  0000 C CNN
-F 3 "" H 4730 3660 50  0000 C CNN
-	1    4730 3660
-	1    0    0    -1
-$EndComp
-$Comp
-L XO-14S X?
+L XO-14S X1
 U 1 1 576A1F0F
 P 8550 4740
-F 0 "X?" H 8310 5100 60  0000 C CNN
+F 0 "X1" H 8310 5100 60  0000 C CNN
 F 1 "XO-14S" H 8550 4370 60  0000 C CNN
-F 2 "" H 8550 4740 60  0000 C CNN
+F 2 "Oscillators:KXO-200" H 8550 4740 60  0000 C CNN
 F 3 "" H 8550 4740 60  0000 C CNN
 	1    8550 4740
@@
 $EndComp
 $Comp
-L VCC #PWR?
+L VCC #PWR03
 U 1 1 576A1FC6
 P 7950 4550
-F 0 "#PWR?" H 7950 4400 50  0001 C CNN
+F 0 "#PWR03" H 7950 4400 50  0001 C CNN
 F 1 "VCC" H 7950 4700 50  0000 C CNN
 F 2 "" H 7950 4550 50  0000 C CNN
@@
 $EndComp
 $Comp
-L GND #PWR?
+L GND #PWR04
 U 1 1 576A21AC
 P 7950 4930
-F 0 "#PWR?" H 7950 4680 50  0001 C CNN
+F 0 "#PWR04" H 7950 4680 50  0001 C CNN
 F 1 "GND" H 7950 4780 50  0000 C CNN
 F 2 "" H 7950 4930 50  0000 C CNN
@@
 wr
 $Comp
-L VCC #PWR?
+L VCC #PWR05
 U 1 1 576A28D7
 P 4700 4650
-F 0 "#PWR?" H 4700 4500 50  0001 C CNN
+F 0 "#PWR05" H 4700 4500 50  0001 C CNN
 F 1 "VCC" H 4700 4800 50  0000 C CNN
 F 2 "" H 4700 4650 50  0000 C CNN
@@
 $EndComp
 $Comp
-L VCC #PWR?
+L VCC #PWR06
 U 1 1 576A2ABD
 P 4560 4750
-F 0 "#PWR?" H 4560 4600 50  0001 C CNN
+F 0 "#PWR06" H 4560 4600 50  0001 C CNN
 F 1 "VCC" H 4560 4900 50  0000 C CNN
 F 2 "" H 4560 4750 50  0000 C CNN
@@
 	1    0    0    -1
 $EndComp
-Wire Wire Line
-	4790 3560 5000 3560
-Wire Wire Line
-	4730 3660 5000 3660
-Wire Wire Line
-	5000 4660 4700 4660
-Wire Wire Line
-	4700 4660 4700 4650
-Wire Wire Line
-	5000 4760 4560 4760
-Wire Wire Line
-	4560 4760 4560 4750
-Wire Wire Line
-	7000 4960 7000 5160
 Text GLabel 10150 6190 0    60   Input ~ 0
 reset
 Text GLabel 5000 5160 0    60   Input ~ 0
 reset
+Text GLabel 10150 5240 0    60   Input ~ 0
+iorq
+Text GLabel 7980 2980 0    60   Input ~ 0
+iorq
+$Comp
+L serial_bort_interface U100
+U 1 1 5777F6E9
+P 3160 3120
+F 0 "U100" H 3160 3120 60  0000 C CNN
+F 1 "serial_port_interface" H 3160 3120 60  0000 C CNN
+F 2 "kicad:serial_to_usb_large" H 3160 3120 60  0000 C CNN
+F 3 "" H 3160 3120 60  0000 C CNN
+	1    3160 3120
+	1    0    0    -1
+$EndComp
+$Comp
+L GND #PWR07
+U 1 1 5777FCC2
+P 2910 2770
+F 0 "#PWR07" H 2910 2520 50  0001 C CNN
+F 1 "GND" H 2910 2620 50  0000 C CNN
+F 2 "" H 2910 2770 50  0000 C CNN
+F 3 "" H 2910 2770 50  0000 C CNN
+	1    2910 2770
+	-1   0    0    1
+$EndComp
+Text GLabel 7000 2860 2    60   Input ~ 0
+cts
+Text GLabel 2910 2820 0    60   Input ~ 0
+cts
+Text GLabel 7000 4060 2    60   Input ~ 0
+tx
+Text GLabel 2910 2970 0    60   Input ~ 0
+tx
+Text GLabel 7000 3960 2    60   Input ~ 0
+rx
+Text GLabel 2910 2920 0    60   Input ~ 0
+rx
+Text GLabel 7000 3260 2    60   Input ~ 0
+dtr
+Text GLabel 2910 3020 0    60   Input ~ 0
+dtr
+$Comp
+L GND #PWR08
+U 1 1 57781892
+P 6000 5460
+F 0 "#PWR08" H 6000 5210 50  0001 C CNN
+F 1 "GND" H 6000 5310 50  0000 C CNN
+F 2 "" H 6000 5460 50  0000 C CNN
+F 3 "" H 6000 5460 50  0000 C CNN
+	1    6000 5460
+	1    0    0    -1
+$EndComp
+$Comp
+L VCC #PWR09
+U 1 1 57781A45
+P 6000 2060
+F 0 "#PWR09" H 6000 1910 50  0001 C CNN
+F 1 "VCC" H 6000 2210 50  0000 C CNN
+F 2 "" H 6000 2060 50  0000 C CNN
+F 3 "" H 6000 2060 50  0000 C CNN
+	1    6000 2060
+	1    0    0    -1
+$EndComp
+Wire Wire Line
+	5000 4660 4700 4660
+Wire Wire Line
+	4700 4660 4700 4650
+Wire Wire Line
+	4560 4760 5000 4760
+Wire Wire Line
+	4560 4760 4560 4750
+Wire Wire Line
+	7000 4960 7000 5160
+$Comp
+L VCC #PWR010
+U 1 1 576A1DB5
+P 4730 3660
+F 0 "#PWR010" H 4730 3510 50  0001 C CNN
+F 1 "VCC" H 4730 3810 50  0000 C CNN
+F 2 "" H 4730 3660 50  0000 C CNN
+F 3 "" H 4730 3660 50  0000 C CNN
+	1    4730 3660
+	1    0    0    -1
+$EndComp
+Wire Wire Line
+	4730 3660 5000 3660
+Wire Wire Line
+	4790 3560 5000 3560
+$Comp
+L VCC #PWR011
+U 1 1 576A1B73
+P 4790 3560
+F 0 "#PWR011" H 4790 3410 50  0001 C CNN
+F 1 "VCC" H 4790 3710 50  0000 C CNN
+F 2 "" H 4790 3560 50  0000 C CNN
+F 3 "" H 4790 3560 50  0000 C CNN
+	1    4790 3560
+	1    0    0    -1
+$EndComp
+Wire Wire Line
+	5000 4960 4700 4960
+Wire Wire Line
+	4700 4960 4700 4760
+Connection ~ 4700 4760
+$Comp
+L C C1
+U 1 1 57796E04
+P 8380 1090
+F 0 "C1" H 8405 1190 50  0000 L CNN
+F 1 "100nF" H 8405 990 50  0000 L CNN
+F 2 "Capacitors_ThroughHole:C_Disc_D3_P2.5" H 8418 940 50  0000 C CNN
+F 3 "" H 8380 1090 50  0000 C CNN
+	1    8380 1090
+	1    0    0    -1
+$EndComp
+$Comp
+L GND #PWR012
+U 1 1 57796E73
+P 8380 1240
+F 0 "#PWR012" H 8380 990 50  0001 C CNN
+F 1 "GND" H 8380 1090 50  0000 C CNN
+F 2 "" H 8380 1240 50  0000 C CNN
+F 3 "" H 8380 1240 50  0000 C CNN
+	1    8380 1240
+	1    0    0    -1
+$EndComp
+$Comp
+L VCC #PWR013
+U 1 1 57796E99
+P 8380 940
+F 0 "#PWR013" H 8380 790 50  0001 C CNN
+F 1 "VCC" H 8380 1090 50  0000 C CNN
+F 2 "" H 8380 940 50  0000 C CNN
+F 3 "" H 8380 940 50  0000 C CNN
+	1    8380 940
+	1    0    0    -1
+$EndComp
+$Comp
+L C C2
+U 1 1 57797882
+P 8690 1090
+F 0 "C2" H 8715 1190 50  0000 L CNN
+F 1 "100nF" H 8715 990 50  0000 L CNN
+F 2 "Capacitors_ThroughHole:C_Disc_D3_P2.5" H 8728 940 50  0000 C CNN
+F 3 "" H 8690 1090 50  0000 C CNN
+	1    8690 1090
+	1    0    0    -1
+$EndComp
+Wire Wire Line
+	8690 940  8380 940
+Wire Wire Line
+	8690 1240 8380 1240
 $EndSCHEMATC
